Commit message: updated from humble to jazzy

File: phoenixbot_description/urdf/groundbot/gazebo_control.xacro (robot description, xacro)
@@ -1,52 +1,37 @@
 <?xml version="1.0" ?>
 <robot xmlns:xacro="http://ros.org/wiki/xacro">
-<!-- Controls the skid steer robot -->
+    <!-- Gazebo Harmonic native systems replace the Gazebo Classic ROS plugins. -->
     <gazebo>
-        <plugin name="skid_steer_drive_controller" filename="libgazebo_ros_skid_steer_drive.so">
-            <updateRate>100.0</updateRate>
-            <robotNamespace>/</robotNamespace>
-            <leftFrontJoint>front_left_wheel_joint</leftFrontJoint>
-            <rightFrontJoint>front_right_wheel_joint</rightFrontJoint>
-            <leftRearJoint>rear_left_wheel_joint</leftRearJoint>
-            <rightRearJoint>rear_right_wheel_joint</rightRearJoint>
-            <wheelSeparation>1.37</wheelSeparation>
-            <wheelDiameter>0.215</wheelDiameter>
-            <robotBaseFrame>base_link</robotBaseFrame>
-            <torque>20</torque>
-            <topicName>cmd_vel</topicName>
-            <broadcastTF>false</broadcastTF>
-        </plugin>
-        <plugin name='skid_steer_drive' filename='libgazebo_ros_diff_drive.so'>
-            <ros>
-            <!-- Set namespace -->
-            <namespace>/</namespace>
-            <!-- Remap default topics -->
-            <!-- <remapping>cmd_vel:=cmd_demo</remapping>
-            <remapping>odom:=odom_demo</remapping> -->
-            </ros>
-            <!-- Update rate -->
-            <update_rate>500</update_rate>
-            <!-- Number of wheel pairs -->
-            <num_wheel_pairs>2</num_wheel_pairs>
-            <!-- wheels0 -->
-            <left_joint>front_left_wheel_joint</left_joint>
-            <right_joint>front_right_wheel_joint</right_joint>
-            <!-- wheels1-->
-            <left_joint>rear_left_wheel_joint</left_joint>
-            <right_joint>rear_right_wheel_joint</right_joint>
-            <!-- kinematics -->
-            <wheel_separation>1.37</wheel_separation>
-            <wheel_separation>1.37</wheel_separation>
-            <wheel_diameter>0.25</wheel_diameter>
-            <wheel_diameter>0.25</wheel_diameter>
-            <!-- limits -->
-            <max_wheel_torque>20</max_wheel_torque>
-            <max_wheel_acceleration>1.0</max_wheel_acceleration>
-            <!-- output -->
-            <publish_odom>true</publish_odom>
-            <publish_odom_tf>true</publish_odom_tf>
-            <publish_wheel_tf>true</publish_wheel_tf>
-            <odometry_frame>odom</odometry_frame>
-            <robot_base_frame>base_link</robot_base_frame>
+      <plugin filename="gz-sim-diff-drive-system"
+              name="gz::sim::systems::DiffDrive">
+        <left_joint>front_left_wheel_joint</left_joint>
+        <left_joint>rear_left_wheel_joint</left_joint>
+        <right_joint>front_right_wheel_joint</right_joint>
+        <right_joint>rear_right_wheel_joint</right_joint>
+        <wheel_separation>1.36</wheel_separation>
+        <wheel_radius>0.125</wheel_radius>
+        <max_linear_acceleration>1.0</max_linear_acceleration>
+        <min_linear_acceleration>-1.0</min_linear_acceleration>
+        <max_angular_acceleration>2.0</max_angular_acceleration>
+        <min_angular_acceleration>-2.0</min_angular_acceleration>
+        <max_linear_velocity>1.0</max_linear_velocity>
+        <min_linear_velocity>-1.0</min_linear_velocity>
+        <max_angular_velocity>1.5</max_angular_velocity>
+        <min_angular_velocity>-1.5</min_angular_velocity>
+        <topic>cmd_vel</topic>
+        <odom_topic>odom</odom_topic>
+        <tf_topic>tf</tf_topic>
+        <frame_id>odom</frame_id>
+        <child_frame_id>base_link</child_frame_id>
+        <odom_publish_frequency>30</odom_publish_frequency>
+      </plugin>
+      <plugin filename="gz-sim-joint-state-publisher-system"
+              name="gz::sim::systems::JointStatePublisher">
+        <joint_name>front_left_wheel_joint</joint_name>
+        <joint_name>front_right_wheel_joint</joint_name>
+        <joint_name>rear_left_wheel_joint</joint_name>
+        <joint_name>rear_right_wheel_joint</joint_name>
+        <topic>joint_states</topic>
+        <update_rate>30</update_rate>
       </plugin>
     </gazebo>

File: phoenixbot_description/urdf/groundbot/phoenixbot_core.xacro (robot description, xacro)
@@ -46,4 +46,7 @@
                 <mesh filename="package://phoenixbot_description/meshes/wheel-motor-assy.dae"/>
             </geometry>
+           <material name="wheel_motor_dark">
+             <color rgba="0.24 0.24 0.26 1" />
+           </material>
          </visual>
          <inertial>
@@ -65,4 +68,7 @@
                 <mesh filename="package://phoenixbot_description/meshes/wheel-motor-assy.dae"/>
             </geometry>
+           <material name="wheel_motor_dark">
+             <color rgba="0.24 0.24 0.26 1" />
+           </material>
          </visual>
          <inertial>
@@ -84,4 +90,7 @@
                 <mesh filename="package://phoenixbot_description/meshes/wheel-motor-assy.dae"/>
             </geometry>
+           <material name="wheel_motor_dark">
+             <color rgba="0.24 0.24 0.26 1" />
+           </material>
          </visual>
          <inertial>
@@ -103,4 +112,7 @@
                 <mesh filename="package://phoenixbot_description/meshes/wheel-motor-assy.dae"/>
             </geometry>
+           <material name="wheel_motor_dark">
+             <color rgba="0.24 0.24 0.26 1" />
+           </material>
          </visual>
          <inertial>

File: phoenixbot_description/urdf/groundbot/robot_cameras.xacro (robot description, xacro)
@@ -17,4 +17,7 @@
           <mesh filename="package://phoenixbot_description/meshes/ZED2.dae"/>
         </geometry>
+        <material name="zed2_shell">
+          <color rgba="0.18 0.20 0.22 1" />
+        </material>
       </visual>
       <collision>
@@ -33,4 +36,6 @@
     <gazebo reference="front_camera">
       <sensor type="camera" name="front_camera">
+        <topic>front_camera/image_raw</topic>
+        <gz_frame_id>front_camera</gz_frame_id>
         <always_on>true</always_on>
         <update_rate>30.0</update_rate>
@@ -60,17 +65,6 @@
             <center>0.5 0.5</center>
           </distortion>
+          <camera_info_topic>front_camera/camera_info</camera_info_topic>
         </camera>
-        <plugin name="front_camera_controller" filename="libgazebo_ros_camera.so">
-          <!-- <robotNamespace>${robot_ns}</robotNamespace> -->
-          <cameraName>front_camera</cameraName>
-          <imageTopicName>image_raw</imageTopicName>
-          <cameraInfoTopicName>camera_info</cameraInfoTopicName>
-          <frameName>camera_optical_frame</frameName>
-          <distortionK1>-0.279817</distortionK1>
-          <distortionK2>0.060321</distortionK2>
-          <distortionK3>0.000487</distortionK3>
-          <distortionT1>0.000310</distortionT1>
-          <distortionT2>0.000000</distortionT2>
-        </plugin>
       </sensor>
     </gazebo>
@@ -91,4 +85,7 @@
           <mesh filename="package://phoenixbot_description/meshes/ZED2.dae"/>
         </geometry>
+        <material name="zed2_shell">
+          <color rgba="0.18 0.20 0.22 1" />
+        </material>
       </visual>
       <collision>
@@ -107,4 +104,6 @@
     <gazebo reference="rear_camera">
       <sensor type="camera" name="rear_camera">
+        <topic>rear_camera/image_raw</topic>
+        <gz_frame_id>rear_camera</gz_frame_id>
         <always_on>true</always_on>
         <update_rate>30.0</update_rate>
@@ -134,17 +133,6 @@
             <center>0.5 0.5</center>
           </distortion>
+          <camera_info_topic>rear_camera/camera_info</camera_info_topic>
         </camera>
-        <plugin name="rear_camera_controller" filename="libgazebo_ros_camera.so">
-          <!-- <robotNamespace>${robot_ns}</robotNamespace> -->
-          <cameraName>rear_camera</cameraName>
-          <imageTopicName>image_raw</imageTopicName>
-          <cameraInfoTopicName>camera_info</cameraInfoTopicName>
-          <frameName>camera_optical_frame</frameName>
-          <distortionK1>-0.279817</distortionK1>
-          <distortionK2>0.060321</distortionK2>
-          <distortionK3>0.000487</distortionK3>
-          <distortionT1>0.000310</distortionT1>
-          <distortionT2>0.000000</distortionT2>
-        </plugin>
       </sensor>
     </gazebo>
@@ -165,4 +153,7 @@
           <mesh filename="package://phoenixbot_description/meshes/ZED2.dae"/>
         </geometry>
+        <material name="zed2_shell">
+          <color rgba="0.18 0.20 0.22 1" />
+        </material>
       </visual>
       <collision>
@@ -181,4 +172,6 @@
     <gazebo reference="downward_camera">
       <sensor type="camera" name="downward_camera">
+        <topic>downward_camera/image_raw</topic>
+        <gz_frame_id>downward_camera</gz_frame_id>
         <always_on>true</always_on>
         <update_rate>30.0</update_rate>
@@ -208,17 +201,6 @@
             <center>0.5 0.5</center>
           </distortion>
+          <camera_info_topic>downward_camera/camera_info</camera_info_topic>
         </camera>
-        <plugin name="downward_camera_controller" filename="libgazebo_ros_camera.so">
-          <!-- <robotNamespace>${robot_ns}</robotNamespace> -->
-          <cameraName>downward_camera</cameraName>
-          <imageTopicName>image_raw</imageTopicName>
-          <cameraInfoTopicName>camera_info</cameraInfoTopicName>
-          <frameName>camera_optical_frame</frameName>
-          <distortionK1>-0.279817</distortionK1>
-          <distortionK2>0.060321</distortionK2>
-          <distortionK3>0.000487</distortionK3>
-          <distortionT1>0.000310</distortionT1>
-          <distortionT2>0.000000</distortionT2>
-        </plugin>
       </sensor>
     </gazebo>

File: phoenixbot_description/urdf/groundbot/ydlidar.xacro (robot description, xacro)
@@ -12,7 +12,7 @@
         <origin xyz="0 0 0" rpy="0 0 0" />
         <geometry>
-          <mesh filename="package://phoenixbot_description//meshes/ydlidar.dae" />
+          <mesh filename="package://phoenixbot_description/meshes/ydlidar.dae" />
         </geometry>
-        <material name="">
+        <material name="ydlidar_body">
           <color rgba="0.64706 0.61961 0.58824 1" />
         </material>
@@ -44,9 +44,12 @@
     </joint>
     <gazebo reference="${name}_link">
-      <sensor type="ray" name="${name}_sensor">
+      <sensor type="gpu_lidar" name="${name}_sensor">
         <pose>0 0 0 0 0 0</pose>
+        <topic>scan</topic>
+        <gz_frame_id>${name}_link</gz_frame_id>
         <visualize>false</visualize>
+        <always_on>true</always_on>
         <update_rate>40</update_rate>
-        <ray>
+        <lidar>
           <scan>
             <horizontal>
@@ -67,12 +70,5 @@
             <stddev>0.01</stddev>
           </noise>
-        </ray>
-        <plugin name="gazebo_ros_${name}_controller" filename="libgazebo_ros_ray_sensor.so">
-          <ros>
-              <remapping>~/out:=scan</remapping>
-          </ros>
-          <output_type>sensor_msgs/LaserScan</output_type>
-          <frameName>${name}_link</frameName>
-        </plugin>
+        </lidar>
       </sensor>
     </gazebo>

File: phoenixbot_description/urdf/groundbot/zed2_camera.xacro (robot description, xacro)
@@ -93,5 +93,8 @@
         <update_rate>30.0</update_rate>
         <visualize>false</visualize>
+        <topic>zed2/center/image_raw</topic>
+        <gz_frame_id>zed2_camera_center</gz_frame_id>
         <camera name="zed2_center_camera">
+          <camera_info_topic>zed2/center/camera_info</camera_info_topic>
           <horizontal_fov>1.9</horizontal_fov>
           <image>
@@ -118,16 +121,4 @@
           </distortion>
         </camera>
-        <plugin name="camera_controller" filename="libgazebo_ros_camera.so">
-          <!-- <robotNamespace>${robot_ns}</robotNamespace> -->
-          <cameraName>camera</cameraName>
-          <imageTopicName>image_raw</imageTopicName>
-          <cameraInfoTopicName>camera_info</cameraInfoTopicName>
-          <frameName>camera_optical_frame</frameName>
-          <distortionK1>-0.279817</distortionK1>
-          <distortionK2>0.060321</distortionK2>
-          <distortionK3>0.000487</distortionK3>
-          <distortionT1>0.000310</distortionT1>
-          <distortionT2>0.000000</distortionT2>
-        </plugin>
       </sensor>
     </gazebo>
@@ -139,5 +130,8 @@
         <update_rate>15.0</update_rate>
         <visualize>false</visualize>
+        <topic>zed2/left_raw/image_raw</topic>
+        <gz_frame_id>zed2_left_camera_optical_frame</gz_frame_id>
         <camera name="zed2_left_raw">
+          <camera_info_topic>zed2/left_raw/camera_info</camera_info_topic>
           <horizontal_fov>1.7633</horizontal_fov>
           <image>
@@ -165,20 +159,4 @@
           </distortion>
         </camera>
-        <plugin name="camera_controller" filename="libgazebo_ros_camera.so">
-          <!-- <robotNamespace>${robot_ns}</robotNamespace> -->
-          <cameraName>zed2/left_raw</cameraName>
-          <imageTopicName>image_raw_color</imageTopicName>
-          <cameraInfoTopicName>camera_info</cameraInfoTopicName>
-          <frameName>zed2_left_camera_optical_frame</frameName>
-          <distortionK1>-0.043693598</distortionK1>
-          <distortionK2>0.0146164996</distortionK2>
-          <distortionT1>-0.006573319</distortionT1>
-          <distortionT2>-0.000216900</distortionT2>
-          <distortionK3>0.000084328</distortionK3>
-          <CxPrime>648.5</CxPrime>
-          <Cx>648.5</Cx>
-          <Cy>366.8340148925781</Cy>
-          <hackBaseline>0.0</hackBaseline>
-        </plugin>
       </sensor>
       <sensor type="depth" name="zed2_left_camera">
@@ -187,38 +165,26 @@
         <update_rate>15.0</update_rate>
         <visualize>false</visualize>
+        <topic>zed2/depth/image_raw</topic>
+        <gz_frame_id>zed2_left_camera_optical_frame</gz_frame_id>
         <camera name="zed2_left">
-          <horizontal_fov>1.7633</horizontal_fov>
-          <image>
-            <width>1280</width>
-            <height>720</height>
-            <format>R8G8B8</format>
-          </image>
-          <clip>
-            <near>0.02</near>
-            <far>300</far>
-          </clip>
-          <noise>
-            <type>gaussian</type>
-            <mean>0.0</mean>
-            <stddev>0.007</stddev>
-          </noise>
-        </camera>
-        <plugin name="camera_controller" filename="libgazebo_ros_openni_kinect.so">
-          <!-- <robotNamespace>${robot_ns}</robotNamespace> -->
-          <cameraName>zed2</cameraName>
-          <imageTopicName>left/image_rect_color</imageTopicName>
-          <cameraInfoTopicName>left/camera_info</cameraInfoTopicName>
-          <depthImageTopicName>depth/depth_registered</depthImageTopicName>
-          <depthImageInfoTopicName>depth/camera_info</depthImageInfoTopicName>
-          <pointCloudTopicName>point_cloud/cloud_registered</pointCloudTopicName>
-          <pointCloudCutoff>0.3</pointCloudCutoff>
-          <pointCloudCutoffMax>20.0</pointCloudCutoffMax>
-          <frameName>zed2_left_camera_optical_frame</frameName>
-          <baseline>0.12</baseline>
-          <CxPrime>658.8206787109375</CxPrime>
-          <Cx>658.8206787109375</Cx>
-          <Cy>372.25787353515625</Cy>
-          <hackBaseline>0.0</hackBaseline>
-        </plugin>
+          <camera_info_topic>zed2/depth/camera_info</camera_info_topic>
+          <horizontal_fov>1.7633</horizontal_fov>
+          <image>
+            <width>1280</width>
+            <height>720</height>
+            <format>R8G8B8</format>
+          </image>
+          <depth_camera>
+            <clip>
+              <near>0.02</near>
+              <far>300</far>
+            </clip>
+          </depth_camera>
+          <noise>
+            <type>gaussian</type>
+            <mean>0.0</mean>
+            <stddev>0.007</stddev>
+          </noise>
+        </camera>
       </sensor>
     </gazebo>
@@ -230,5 +196,8 @@
         <update_rate>15.0</update_rate>
         <visualize>false</visualize>
+        <topic>zed2/right_raw/image_raw</topic>
+        <gz_frame_id>zed2_right_camera_optical_frame</gz_frame_id>
         <camera name="zed2_right_raw">
+          <camera_info_topic>zed2/right_raw/camera_info</camera_info_topic>
           <horizontal_fov>1.7633</horizontal_fov>
           <image>
@@ -255,20 +224,4 @@
           </distortion>
         </camera>
-        <plugin name="camera_controller" filename="libgazebo_ros_camera.so">
-          <!-- <robotNamespace>${robot_ns}</robotNamespace> -->
-          <cameraName>zed2/right_raw</cameraName>
-          <imageTopicName>image_raw_color</imageTopicName>
-          <cameraInfoTopicName>camera_info</cameraInfoTopicName>
-          <frameName>zed2_right_camera_optical_frame</frameName>
-          <distortionK1>-0.040993299</distortionK1>
-          <distortionK2>0.009593590</distortionK2>
-          <distortionT1>-0.004429849</distortionT1>
-          <distortionT2>0.000192024</distortionT2>
-          <distortionK3>-0.000320880</distortionK3>
-          <CxPrime>659.3049926757812</CxPrime>
-          <Cx>659.3049926757812</Cx>
-          <Cy>371.39849853515625</Cy>
-          <hackBaseline>0.12</hackBaseline>
-        </plugin>
       </sensor>
       <sensor type="camera" name="zed2_right_camera">
@@ -277,32 +230,24 @@
         <update_rate>15.0</update_rate>
         <visualize>false</visualize>
+        <topic>zed2/right/image_raw</topic>
+        <gz_frame_id>zed2_right_camera_optical_frame</gz_frame_id>
         <camera name="zed2_right">
-          <horizontal_fov>1.7633</horizontal_fov>
-          <image>
-            <width>1280</width>
-            <height>720</height>
-            <format>R8G8B8</format>
-          </image>
-          <clip>
-            <near>0.02</near>
-            <far>300</far>
-          </clip>
-          <noise>
-            <type>gaussian</type>
-            <mean>0.0</mean>
-            <stddev>0.007</stddev>
-          </noise>
-        </camera>
-        <plugin name="camera_controller" filename="libgazebo_ros_camera.so">
-          <!-- <robotNamespace>${robot_ns}</robotNamespace> -->
-          <cameraName>zed2/right</cameraName>
-          <imageTopicName>image_rect_color</imageTopicName>
-          <cameraInfoTopicName>camera_info</cameraInfoTopicName>
-          <frameName>zed2_right_camera_optical_frame</frameName>
-          <CxPrime>658.8206787109375</CxPrime>
-          <Cx>658.8206787109375</Cx>
-          <Cy>372.25787353515625</Cy>
-          <hackBaseline>0.12</hackBaseline>
-        </plugin>
+          <camera_info_topic>zed2/right/camera_info</camera_info_topic>
+          <horizontal_fov>1.7633</horizontal_fov>
+          <image>
+            <width>1280</width>
+            <height>720</height>
+            <format>R8G8B8</format>
+          </image>
+          <clip>
+            <near>0.02</near>
+            <far>300</far>
+          </clip>
+          <noise>
+            <type>gaussian</type>
+            <mean>0.0</mean>
+            <stddev>0.007</stddev>
+          </noise>
+        </camera>
       </sensor>
     </gazebo>
@@ -310,16 +255,7 @@
     <gazebo reference="zed2_left_camera_frame">
       <sensor type="imu" name="zed2_imu_sensor">
+        <topic>zed2/imu/data</topic>
+        <gz_frame_id>zed2_left_camera_frame</gz_frame_id>
         <update_rate>100</update_rate>
-        <plugin filename="libgazebo_ros_imu_sensor.so" name="imu_plugin">
-          <!-- <robotNamespace>${robot_ns}</robotNamespace> -->
-          <topicName>zed2/imu/data</topicName>
-          <frameName>zed2_imu_link</frameName>
-          <updateRateHZ>100.0</updateRateHZ>
-          <gaussianNoise>0.01</gaussianNoise>
-          <initialOrientationAsReference>false</initialOrientationAsReference>
-          <!-- IMU frame offset copied from an actual ZED2 camera -->
-          <xyzOffset>-0.002 -0.023 -0.002</xyzOffset>
-          <rpyOffset>0.0014025 -0.0000012 -0.0016915</rpyOffset>
-        </plugin>
       </sensor>
     </gazebo>
