Commit message: updated files to work with gps and kiwirover

File: phoenixbot_description/urdf/groundbot/phoenixbot.xacro (robot description, xacro)
@@ -8,5 +8,4 @@
     <xacro:include filename="$(find phoenixbot_description)/urdf/groundbot/ydlidar.xacro" />
     <xacro:include filename="$(find phoenixbot_description)/urdf/groundbot/zed2_camera.xacro" />
-    <!-- <xacro:include filename="$(find phoenixbot_description)/urdf/gps.xacro" /> -->
     <xacro:include filename="robot_cameras.xacro"/>
     <!-- ydlidar -->
@@ -15,7 +14,29 @@
     </xacro:ydlidar_sensor>
     <!-- gps -->
-    <!-- <xacro:gps_sensor parent="base_link">
-        <origin xyz="0 0 0.2" rpy="0 0 0"/>
-    </xacro:gps_sensor> -->
+    <link name="gps_link"/>
+    <joint name="gps_joint" type="fixed">
+      <parent link="base_link"/>
+      <child link="gps_link"/>
+      <origin xyz="-0.05 0 0.05" rpy="0 0 0"/>
+    </joint>
+    <gazebo reference="gps_link">
+      <sensor name="navsat" type="navsat">
+        <always_on>true</always_on>
+        <update_rate>1</update_rate>
+        <topic>/gps/fix</topic>
+        <gz_frame_id>gps_link</gz_frame_id>
+        <navsat>
+        </navsat>
+      </sensor>
+    </gazebo>
+    <gazebo reference="chassis">
+      <sensor name="imu_sensor" type="imu">
+        <always_on>true</always_on>
+        <update_rate>50</update_rate>
+        <topic>/imu/data</topic>
+        <gz_frame_id>chassis</gz_frame_id>
+        <imu/>
+      </sensor>
+    </gazebo>
     <!-- front_camera -->
     <xacro:front_camera parent="chassis">
